File: KiCAD/Drive/Drive.kicad_pcb (KiCad board)
At the start: 2 copper layers, 95 x 65 mm, 85 parts, among them J3.3 Conn_01x03_Pin, U15-5 DC-DC Converter, U2 LM324, U30-15 DC-DC Converter

Commit message: design bug fix
Routing:
- net -30: track 81.5 -> 91.6 mm, vias 31 -> 36
- net /NU: track 12.6 -> 16.2 mm
Changed lines of the file:
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@@
   (segment (start 160.4625 56.5375) (end 160.5 56.5) (width 0.5) (layer "F.Cu") (net 2))
   (segment (start 171 82.9875) (end 170.9625 82.95) (width 0.5) (layer "F.Cu") (net 2))
+  (segment (start 104.075 93) (end 105.075 92) (width 0.2) (layer "F.Cu") (net 2))
   (segment (start 160.5 95.5) (end 162 97) (width 0.5) (layer "F.Cu") (net 2))
   (segment (start 115.5 57.5) (end 117.55 57.5) (width 0.5) (layer "F.Cu") (net 2))
@@
   (segment (start 108.55 74.5) (end 107.05 73) (width 0.5) (layer "F.Cu") (net 2))
   (segment (start 172.485 96.425) (end 175 98.94) (width 2) (layer "F.Cu") (net 2))
+  (segment (start 103.95 77) (end 105.5 77) (width 0.2) (layer "F.Cu") (net 2))
   (segment (start 144.5 66) (end 144.5 66.575) (width 0.5) (layer "F.Cu") (net 2))
   (segment (start 174.9625 72.4) (end 174.9625 71.4625) (width 0.5) (layer "F.Cu") (net 2))
   (segment (start 110.5 76.45) (end 108.55 74.5) (width 0.5) (layer "F.Cu") (net 2))
+  (segment (start 104 81) (end 105.5 81) (width 0.2) (layer "F.Cu") (net 2))
   (segment (start 147.5 110.5) (end 150 108) (width 0.5) (layer "F.Cu") (net 2))
   (segment (start 148.55 59) (end 150.5 59) (width 0.5) (layer "F.Cu") (net 2))
   (segment (start 144 110.5) (end 147.5 110.5) (width 0.5) (layer "F.Cu") (net 2))
   (segment (start 110.5 77) (end 110.5 76.45) (width 0.5) (layer "F.Cu") (net 2))
+  (segment (start 103.95 89) (end 105 89) (width 0.2) (layer "F.Cu") (net 2))
   (segment (start 175 98.94) (end 175 100.5) (width 2) (layer "F.Cu") (net 2))
   (segment (start 170.05 68.55) (end 168.5 67) (width 0.5) (layer "F.Cu") (net 2))
+  (segment (start 105.5 77) (end 106 77.5) (width 0.2) (layer "F.Cu") (net 2))
   (segment (start 123 61.075) (end 123 59) (width 0.5) (layer "F.Cu") (net 2))
   (segment (start 118.5 67) (end 120 67) (width 0.5) (layer "F.Cu") (net 2))
@@
   (segment (start 107 73) (end 103.95 73) (width 0.5) (layer "F.Cu") (net 2))
   (segment (start 137.45 66) (end 144.5 66) (width 0.5) (layer "F.Cu") (net 2))
+  (segment (start 105.075 92) (end 106 92) (width 0.2) (layer "F.Cu") (net 2))
   (segment (start 147.5 64) (end 146.425 64) (width 0.5) (layer "F.Cu") (net 2))
   (segment (start 127 110.5) (end 128.5 110.5) (width 0.5) (layer "F.Cu") (net 2))
   (segment (start 149.5 69.1) (end 149.5 70.5) (width 0.5) (layer "F.Cu") (net 2))
+  (segment (start 105.5 81) (end 106 81.5) (width 0.2) (layer "F.Cu") (net 2))
   (segment (start 165.9625 64.4625) (end 166.5 65) (width 0.5) (layer "F.Cu") (net 2))
   (segment (start 160.4625 58.55) (end 160.4625 56.5375) (width 0.5) (layer "F.Cu") (net 2))
@@
   (segment (start 121.575 68.45) (end 121.45 68.45) (width 0.5) (layer "F.Cu") (net 2))
   (segment (start 172.485 93) (end 172.485 96.425) (width 2) (layer "F.Cu") (net 2))
+  (segment (start 105 89) (end 105.5 88.5) (width 0.2) (layer "F.Cu") (net 2))
+  (segment (start 104 85) (end 105.5 85) (width 0.2) (layer "F.Cu") (net 2))
   (segment (start 121.45 68.45) (end 120 67) (width 0.5) (layer "F.Cu") (net 2))
   (segment (start 162 97) (end 162.5 97) (width 0.5) (layer "F.Cu") (net 2))
@@
   (via (at 148 63.5) (size 0.8) (drill 0.4) (layers "F.Cu" "B.Cu") (net 2))
   (via (at 154.5 108) (size 0.8) (drill 0.4) (layers "F.Cu" "B.Cu") (free) (net 2))
+  (via (at 106 81.5) (size 0.8) (drill 0.4) (layers "F.Cu" "B.Cu") (free) (net 2))
   (via (at 120 67) (size 0.8) (drill 0.4) (layers "F.Cu" "B.Cu") (free) (net 2))
   (via (at 107 73) (size 0.8) (drill 0.4) (layers "F.Cu" "B.Cu") (net 2))
@@
   (via (at 171 85) (size 0.8) (drill 0.4) (layers "F.Cu" "B.Cu") (free) (net 2))
   (via (at 151.5 106.5) (size 0.8) (drill 0.4) (layers "F.Cu" "B.Cu") (free) (net 2))
+  (via (at 105.5 88.5) (size 0.8) (drill 0.4) (layers "F.Cu" "B.Cu") (free) (net 2))
   (via (at 153 108) (size 0.8) (drill 0.4) (layers "F.Cu" "B.Cu") (free) (net 2))
+  (via (at 106 92) (size 0.8) (drill 0.4) (layers "F.Cu" "B.Cu") (free) (net 2))
   (via (at 150 106.5) (size 0.8) (drill 0.4) (layers "F.Cu" "B.Cu") (free) (net 2))
   (via (at 155 111) (size 0.8) (drill 0.4) (layers "F.Cu" "B.Cu") (free) (net 2))
@@
   (via (at 168.5 67) (size 0.8) (drill 0.4) (layers "F.Cu" "B.Cu") (net 2))
   (via (at 153 105) (size 0.8) (drill 0.4) (layers "F.Cu" "B.Cu") (free) (net 2))
+  (via (at 105.5 85) (size 0.8) (drill 0.4) (layers "F.Cu" "B.Cu") (free) (net 2))
   (via (at 150 108) (size 0.8) (drill 0.4) (layers "F.Cu" "B.Cu") (free) (net 2))
   (via (at 160.5 56.5) (size 0.8) (drill 0.4) (layers "F.Cu" "B.Cu") (free) (net 2))
   (via (at 153 106.5) (size 0.8) (drill 0.4) (layers "F.Cu" "B.Cu") (free) (net 2))
+  (via (at 106 77.5) (size 0.8) (drill 0.4) (layers "F.Cu" "B.Cu") (free) (net 2))
   (segment (start 107 93) (end 105 95) (width 0.3) (layer "F.Cu") (net 3))
   (segment (start 108.545 89.455) (end 107 91) (width 0.3) (layer "F.Cu") (net 3))
@@
   (segment (start 98.95 77) (end 101 77) (width 0.3) (layer "F.Cu") (net 7))
   (segment (start 98.875 73) (end 101 73) (width 0.3) (layer "F.Cu") (net 8))
-  (segment (start 104.5 75) (end 102 75) (width 0.3) (layer "F.Cu") (net 8))
+  (segment (start 102 75) (end 101 74) (width 0.3) (layer "F.Cu") (net 8))
+  (segment (start 105 75) (end 102 75) (width 0.3) (layer "F.Cu") (net 8))
+  (segment (start 108 78) (end 105 75) (width 0.3) (layer "F.Cu") (net 8))
+  (segment (start 109.455 81.455) (end 108 80) (width 0.3) (layer "F.Cu") (net 8))
+  (segment (start 108 80) (end 108 78) (width 0.3) (layer "F.Cu") (net 8))
+  (segment (start 121.7 81.455) (end 109.455 81.455) (width 0.3) (layer "F.Cu") (net 8))
   (segment (start 101 74) (end 101 73) (width 0.3) (layer "F.Cu") (net 8))
-  (segment (start 102 75) (end 101 74) (width 0.3) (layer "F.Cu") (net 8))
-  (segment (start 106 76.5) (end 104.5 75) (width 0.3) (layer "F.Cu") (net 8))
-  (segment (start 109.455 81.455) (end 106 78) (width 0.3) (layer "F.Cu") (net 8))
-  (segment (start 106 78) (end 106 76.5) (width 0.3) (layer "F.Cu") (net 8))
-  (segment (start 121.7 81.455) (end 109.455 81.455) (width 0.3) (layer "F.Cu") (net 8))
   (segment (start 115.5 79.05) (end 115.5 79.855) (width 0.3) (layer "F.Cu") (net 9))
   (segment (start 113.45 77) (end 115.5 79.05) (width 0.3) (layer "F.Cu") (net 9))
@@
   (segment (start 152.5 85) (end 151.5 84) (width 0.3) (layer "F.Cu") (net 49))
   (segment (start 156.575 85) (end 152.5 85) (width 0.3) (layer "F.Cu") (net 49))
+  (segment (start 157.5 89.5) (end 157.5 86.075) (width 0.25) (layer "F.Cu") (net 49))
   (segment (start 157.575 86) (end 156.575 85) (width 0.3) (layer "F.Cu") (net 49))
   (segment (start 151.405 82.405) (end 151.5 82.5) (width 2) (layer "F.Cu") (net 49))
+  (segment (start 157.5 86.075) (end 157.575 86) (width 0.25) (layer "F.Cu") (net 49))
   (segment (start 135.5 107.675) (end 135.6 107.575) (width 0.3) (layer "F.Cu") (net 51))
   (segment (start 133.1 107.675) (end 135.5 107.675) (width 0.3) (layer "F.Cu") (net 51))
